File: PCB/Turntable/iidx_tt.kicad_pcb (KiCad board)
At the start: 2 copper layers, 63.5 x 23 mm, 8 parts, among them J1 Conn_01x05_Female, J2 Conn_01x03_Female, U1 AS5600

Commit message: Update turntable PCB
Parts:
- moved J1 4.00 mm to (223.8, 97.5)
- moved J2 1.00 mm to (235.8, 97.5)
Routing:
- net Net-(R1-Pad2): track 25.0 -> 29.2 mm
- net Net-(R2-Pad2): track 26.0 -> 30.0 mm
- net GND: track 15.2 -> 11.9 mm, vias 2 -> 4
- net Net-(J1-Pad2): track 6.25 -> 3.25 mm
Other:
- outline, holes or cut-outs redrawn
