File: PCB/Pico/iidx_pico.kicad_pcb (KiCad board)
At the start: 2 copper layers, 180 x 160 mm, 77 parts, among them J1 Spin, J2 Spin, J3 RGB, J4 RGB, J5 Spin, J6 Spin, SW1 SWITCH_SPST, SW10 SWITCH_SPST, SW11 SWITCH_SPST, SW12 Tact_4pin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

Commit message: Pico PCB v1.42 for lenient stabilizer cut
Parts:
- moved D43 0.20 mm to (145.6, 100.4)
- moved D44 0.20 mm to (145.6, 76.4)
- moved D53 0.20 mm to (166.1, 156.4)
- moved D54 0.20 mm to (166.1, 132.4)
- moved D63 0.20 mm to (186.6, 100.4)
- moved D64 0.20 mm to (186.6, 76.4)
- moved D73 0.20 mm to (207.1, 156.4)
- moved D74 0.20 mm to (207.1, 132.4)
- moved D11 0.20 mm to (67.5, 156.4)
- moved D12 0.20 mm to (67.5, 132.4)
- moved D13 0.20 mm to (84.1, 156.4)
- moved D14 0.20 mm to (84.1, 132.4)
- moved D21 0.20 mm to (88.0, 100.4)
- moved D22 0.20 mm to (88.0, 76.4)
- moved D23 0.20 mm to (104.6, 100.4)
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Routing:
- net +5V: track 1136.0 -> 1140.8 mm
- net /LED7: track 142.1 -> 143.5 mm
- net /LED2: track 97.1 -> 98.4 mm
- net /LED5: track 114.8 -> 115.8 mm
- net /LED1: track 114.4 -> 115.4 mm
- net /LED3: track 114.4 -> 115.3 mm
- net /LED6: track 160.1 -> 161.0 mm
- net /LED4: track 160.8 -> 161.4 mm
Other:
- board text added: "IIDX Pico v1.42"
- board text removed: "IIDX Pico v1.41"
