File: PCB/Teeny/iidx_teeny.kicad_pcb (KiCad board)
At the start: 2 copper layers, 150 x 100 mm, 57 parts, among them J1 RGB, J2 RGB, J3 Spin, J4 Spin, J5 Spin, J6 Spin, SW1 SWITCH_SPST, SW10 SWITCH_SPST, SW11 SWITCH_SPST, SW12 SWITCH_SPST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

Commit message: Teeny PCB v1.31, finetune
Parts:
- removed the R1 at (93.4, 101.6)
- removed the R2 at (108.4, 74.2)
- renumbered R20 to R1, R21 to R2
Connections:
- U1 pad 17: Net-(U1-GPIO13) -> /LED2
- U1 pad 34: Net-(U1-GPIO28_ADC2) -> /TT_LED
Routing:
- net /LED2: track 28.5 -> 43.6 mm
- net Net-(U1-GPIO13): track 14.7 -> 0.00 mm
- net Net-(U1-GPIO28_ADC2): track 4.78 -> 0.00 mm
- net /TT_LED: track 179.1 -> 182.8 mm
- net GND: track 63.9 -> 61.7 mm
Other:
- board text added: "IIDX Teeny v1.31"
- board text added: "V G L"
- board text added: "V L G"
- board text removed: "IIDX Teeny v1.3"
