File: PCB/Teeny/iidx_teeny.kicad_pcb (KiCad board)
At the start: 2 copper layers, 150 x 100 mm, 55 parts, among them J1 RGB, J2 RGB, J3 Spin, J4 Spin, J5 Spin, J6 Spin, SW1 SWITCH_SPST, SW10 SWITCH_SPST, SW11 SWITCH_SPST, SW12 SWITCH_SPST, SW13 SWITCH_SPST, SW2 SWITCH_SPST, SW3 SWITCH_SPST, SW4 SWITCH_SPST, SW5 SWITCH_SPST, SW6 SWITCH_SPST, SW7 SWITCH_SPST, SW8 SWITCH_SPST, SW9 SWITCH_SPST, U1 PiPico_No_SWD, U2 TMAG5273, U3 AS5600

Commit message: Teeny PCB v1.4 to support MT6701 sensor
Parts:
- added JP1: DIR, Jumper:SolderJumper-2_P1.3mm_Open_RoundedPad1.0x1.5mm, F.Cu at (76.8, 115.0)
Connections:
- U3 pad 8: GND -> Net-(JP1-A)
Routing:
- net Net-(JP1-A): track 0.00 -> 2.02 mm
- net Net-(U1-GPIO8): track 62.7 -> 63.8 mm
- net GND: track 61.7 -> 62.8 mm
- net /LED8: track 100.1 -> 100.7 mm
Other:
- board text added: "IIDX Teeny v1.4"
- board text added: "github.com/whowechina"
- board text removed: "IIDX Teeny v1.31"
