File: PCB/Teeny/iidx_teeny.kicad_sch (KiCad schematic)
At the start: 55 parts, among them J1 RGB, J2 RGB, J3 Spin, J4 Spin, J5 Spin, J6 Spin, SW1 SWITCH_SPST, SW10 SWITCH_SPST, SW11 SWITCH_SPST, SW12 SWITCH_SPST, SW13 SWITCH_SPST, SW2 SWITCH_SPST, SW3 SWITCH_SPST, SW4 SWITCH_SPST, SW5 SWITCH_SPST, SW6 SWITCH_SPST, SW7 SWITCH_SPST, SW8 SWITCH_SPST, SW9 SWITCH_SPST, U1 PiPico_No_SWD, U2 TMAG5273, U3 AS5600

Commit message: Teeny PCB v1.4 to support MT6701 sensor
Parts:
- added JP1: DIR, Jumper:SolderJumper-2_P1.3mm_Open_RoundedPad1.0x1.5mm, symbol Jumper:SolderJumper_2_Open
Connections:
- net GND: now also JP1.2 (B); no longer U3.8 (DIR)
- new net: JP1.1 (A), U3.8 (DIR)
